File: SteveEsquematico/esquematico_placa.sch (EAGLE design)
At the start: 15 parts, among them T1 NTA4151P, U1 MCP73832T-5ACI/OT

Commit message: Teste
Parts:
- removed C1: 4,7uF x 16V, SCAP-PANASONIC5.5V1F5MM20MM:PANASONIC-SCAP-5.5V-0.1F
- removed C3: 1F x 2.5V, SCAP-PANASONIC5.5V1F5MM20MM:PANASONIC-SCAP-5.5V-0.1F
- C2: value 1F x 2.5V -> 1F x 5.5V
Connections:
- removed net N$3: C2.-, C3.+
- net GND: no longer C1.-
- net OUT+: no longer C1.+
- net VCAP: now also C2.-; no longer C3.-
Other:
- note added: "Bateria de litio"
Changed lines of the file:
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@@
 <setting verticaltext="up"/>
 </settings>
-<grid distance="0.1" unitdist="inch" unit="inch" style="lines" multiple="1" display="no" altdistance="0.01" altunitdist="inch" altunit="inch"/>
+<grid distance="0.01" unitdist="inch" unit="inch" style="lines" multiple="1" display="yes" altdistance="0.01" altunitdist="inch" altunit="inch"/>
 <layers>
 <layer number="1" name="Top" color="4" fill="1" visible="no" active="no"/>
@@
 <part name="FRAME1" library="frames" library_urn="urn:adsk.eagle:library:229" deviceset="A3L-LOC" device=""/>
 <part name="U$1" library="nta4151p" deviceset="NTA4151P" device=""/>
-<part name="C2" library="SCAP-PANASONIC5.5V1F5MM20MM" deviceset="PANASONIC-SCAP-5.5V-0.1F" device="" value="1F x 2.5V"/>
+<part name="C2" library="SCAP-PANASONIC5.5V1F5MM20MM" deviceset="PANASONIC-SCAP-5.5V-0.1F" device="" value="1F x 5.5V"/>
 <part name="GND2" library="supply1" library_urn="urn:adsk.eagle:library:371" deviceset="GND" device=""/>
-<part name="C3" library="SCAP-PANASONIC5.5V1F5MM20MM" deviceset="PANASONIC-SCAP-5.5V-0.1F" device="" value="1F x 2.5V"/>
 <part name="U1" library="MCP73832T-5ACI_OT" deviceset="MCP73832T-5ACI/OT" device=""/>
 <part name="R5" library="0805 Resistor" deviceset="CRGH0805F392R" device="" value="2K R"/>
-<part name="C1" library="SCAP-PANASONIC5.5V1F5MM20MM" deviceset="PANASONIC-SCAP-5.5V-0.1F" device="" value="4,7uF x 16V"/>
 <part name="GND3" library="supply1" library_urn="urn:adsk.eagle:library:371" deviceset="GND" device=""/>
 </parts>
@@
 <text x="25.4" y="98.044" size="3.81" layer="97">LIPO CHARGER</text>
 <text x="342.9" y="20.32" size="1.778" layer="94">Desenhado por Steve Nascimento</text>
+<text x="109.22" y="50.8" size="1.778" layer="95">Bateria de litio</text>
 </plain>
 <instances>
@@
 <attribute name="VALUE" x="43.688" y="117.348" size="1.778" layer="96"/>
 </instance>
-<instance part="C3" gate="G$1" x="117.602" y="122.428" smashed="yes">
-<attribute name="NAME" x="104.902" y="127.508" size="1.27" layer="94"/>
-<attribute name="VALUE" x="104.902" y="117.348" size="1.27" layer="94"/>
-</instance>
 <instance part="U1" gate="A" x="73.66" y="63.5" smashed="yes" rot="R180">
 <attribute name="NAME" x="73.31721875" y="77.216659375" size="2.08845" layer="95" ratio="10" rot="SR180"/>
@@
 <attribute name="NAME" x="72.39" y="44.6786" size="1.778" layer="95"/>
 <attribute name="VALUE" x="69.85" y="50.038" size="1.27" layer="96"/>
-</instance>
-<instance part="C1" gate="G$1" x="35.56" y="45.72" smashed="yes" rot="R270">
-<attribute name="NAME" x="40.64" y="58.42" size="1.27" layer="94" rot="R270"/>
-<attribute name="VALUE" x="30.48" y="58.42" size="1.27" layer="94" rot="R270"/>
 </instance>
 <instance part="GND3" gate="1" x="99.06" y="35.56" smashed="yes">
@@
 <pinref part="U1" gate="A" pin="VDD"/>
 <wire x1="55.88" y1="66.04" x2="35.56" y2="66.04" width="0.1524" layer="91"/>
-<pinref part="C1" gate="G$1" pin="+"/>
 <wire x1="35.56" y1="66.04" x2="35.56" y2="55.88" width="0.1524" layer="91"/>
 <wire x1="35.56" y1="66.04" x2="17.78" y2="66.04" width="0.1524" layer="91"/>
@@
 <pinref part="U1" gate="A" pin="VSS"/>
 <wire x1="99.06" y1="66.04" x2="91.44" y2="66.04" width="0.1524" layer="91"/>
-<pinref part="C1" gate="G$1" pin="-"/>
 <wire x1="35.56" y1="53.34" x2="35.56" y2="38.1" width="0.1524" layer="91"/>
 <wire x1="35.56" y1="38.1" x2="99.06" y2="38.1" width="0.1524" layer="91"/>
@@
 <junction x="99.06" y="38.1"/>
 <pinref part="GND3" gate="1" pin="GND"/>
-<wire x1="121.92" y1="48.26" x2="116.84" y2="48.26" width="0.1524" layer="91"/>
 <wire x1="116.84" y1="48.26" x2="116.84" y2="38.1" width="0.1524" layer="91"/>
+<label x="119.38" y="45.72" size="1.778" layer="95"/>
 </segment>
 </net>
@@
 <junction x="128.016" y="141.732"/>
 <label x="131.064" y="143.256" size="1.27" layer="95"/>
-<pinref part="C3" gate="G$1" pin="-"/>
-<wire x1="109.982" y1="122.428" x2="128.016" y2="122.428" width="0.1524" layer="91"/>
-</segment>
-</net>
-<net name="N$3" class="0">
-<segment>
 <pinref part="C2" gate="G$1" pin="-"/>
-<pinref part="C3" gate="G$1" pin="+"/>
-<wire x1="84.328" y1="122.428" x2="107.442" y2="122.428" width="0.1524" layer="91"/>
+<wire x1="84.328" y1="122.428" x2="128.016" y2="122.428" width="0.1524" layer="91"/>
 </segment>
 </net>
@@
 <wire x1="116.84" y1="68.58" x2="116.84" y2="53.34" width="0.1524" layer="91"/>
 <junction x="116.84" y="68.58"/>
-<wire x1="121.92" y1="53.34" x2="116.84" y2="53.34" width="0.1524" layer="91"/>
 <label x="134.62" y="71.12" size="1.27" layer="95"/>
-</segment>
-</net>
+<label x="119.38" y="55.88" size="1.778" layer="95"/>
+</segment>
+</net>
