File: No_Agricultura/esquematico_placa.sch (EAGLE design)
At the start: 32 parts, among them IC2 PIC18F45K80-I_PT, M1 NTA4151P, M2 NTA4151P, M3 NTA4151P, M4 NTA4151P, U1 HTU21D, X1 BAT, X3 INPUT, X6 PINS I/O

Commit message: Atualizando pasta completa
Parts:
- removed C1, C2: 1F x 2.5V, M0810-2R5105-R:M0810-2R5105-R
- removed LED3: (no value), led:LED5MM
- added IC1: DW01-P, DW01-P:DW01-P
- added IC3: TP4056, TP4056:TP4056
- added Q1: FS8205A, FS8205A:FS8205A
- added R10, R9: 1K R, 0805 Resistor:CRGH0805F392R
- added R8: 1.2K R, 0805 Resistor:CRGH0805F392R
Connections:
- removed net N$8: C1.+, C2.-
- new net N$10: IC3.PROG, R8.2
- new net N$12: IC1.VCC, R10.2
- new net N$15: IC1.CS, R9.2
- new net N$16: IC1.OC, Q1.G2
- new net N$21: IC1.OD, Q1.G1
- new net N$6: IC3.CHRG, LED1.C
- new net N$7: IC3.STDBY, LED2.C
- new net VSSBAT: IC1.GND, Q1.S1_1
- net GND: now also IC3.GND, IC3.TEMP, Q1.S2_2, R8.1, R9.1; no longer C1.-
- net OUT+: now also IC3.CE, IC3.VCC, LED1.A, LED2.A
- net VBAT: now also IC3.BAT, R10.1
- net VCAP: no longer C2.+
Other:
- note removed: "LEDS DE INDICAÇAO"
- moved on the sheet: LED1, LED2
